File: HP9815_OVP_Schematic/HP9815_OVP/HP9815_OVP.kicad_pcb (KiCad board)
At the start: 2 copper layers, 19 parts, among them Q1 600V, 8A, Q2 600V, 8A, Q3 600V, 8A, Q4 600V, 8A, Q5 600V, 8A, U1 TL431DBZ-SOT-23, U2 TL431DBZ-SOT-23, U3 TL431DBZ-SOT-23, U4 TL431DBZ-SOT-23, U5 TL431DBZ-SOT-23

Commit message: Simulated started and outline done
Parts:
- added J1: IPBT-103-H1-T-D-K, DB_Connector_Samtec:SAMTEC_IPBT-103-H1-T-D-K, F.Cu at (139.1, 104.1)
- added J2: IPBT-104-H1-T-D-K, DB_Connector_Samtec:SAMTEC_IPBT-104-H1-T-D-K, F.Cu at (155.6, 104.1)
- moved MH3 198.4 mm to (250.4, 72.9)
- moved MH4 173.3 mm to (250.4, 80.9)
- moved Q1 163.6 mm to (229.1, 44.1)
- moved U1 74.7 mm to (256.9, 68.5)
- moved U2 74.7 mm to (256.9, 73.1)
- moved U3 74.7 mm to (256.9, 77.7)
- moved U4 74.7 mm to (256.9, 82.4)
- moved U5 74.7 mm to (256.9, 87.0)
- moved FH1 74.0 mm to (240.4, 43.3)
- moved FH2 74.0 mm to (240.4, 49.9)
- moved FH3 74.0 mm to (240.4, 56.5)
- moved FH4 74.0 mm to (240.4, 63.0)
- moved FH5 74.0 mm to (240.4, 69.6)
- moved MH1 69.5 mm to (109.7, 92.8)
- moved MH2 65.1 mm to (129.7, 92.8)
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Other:
- board outline added: 84.9 x 77 mm

Commit message: Commit before relinking ref des
Parts:
- removed MH3, MH4: 3mm, DB_Mounting_Holes:MountingHole_3.2mm_M3_Pad
- added C1: 10nF, DB_SMD_Capacitors:C_0603_1608Metric_Pad1.08x0.95mm_HandSolder, F.Cu at (205.8, 32.5)
- added C2: 10nF, DB_SMD_Capacitors:C_0603_1608Metric_Pad1.08x0.95mm_HandSolder, F.Cu at (205.8, 35.0)
- added C3: 10nF, DB_SMD_Capacitors:C_0603_1608Metric_Pad1.08x0.95mm_HandSolder, F.Cu at (205.8, 37.5)
- added C4: 10nF, DB_SMD_Capacitors:C_0603_1608Metric_Pad1.08x0.95mm_HandSolder, F.Cu at (205.8, 40.0)
- added C5: 10nF, DB_SMD_Capacitors:C_0603_1608Metric_Pad1.08x0.95mm_HandSolder, F.Cu at (205.8, 42.5)
- added LD1: Green, DB_SMD_LED:LED_0603_1608Metric_Green_Cath_Dot, F.Cu at (145.2, 63.7)
- added LD2: Green, DB_SMD_LED:LED_0603_1608Metric_Green_Cath_Dot, F.Cu at (137.9, 63.7)
- added LD3: Green, DB_SMD_LED:LED_0603_1608Metric_Green_Cath_Dot, F.Cu at (167.1, 63.7)
- added LD4: Green, DB_SMD_LED:LED_0603_1608Metric_Green_Cath_Dot, F.Cu at (159.8, 63.7)
- added LD5: Green, DB_SMD_LED:LED_0603_1608Metric_Green_Cath_Dot, F.Cu at (152.5, 63.7)
- added Q10: 600V, 8A, Package_TO_SOT_SMD:TO-252-2, F.Cu at (226.3, 162.7)
- added Q6: 600V, 8A, Package_TO_SOT_SMD:TO-252-2, F.Cu at (226.3, 154.5)
- added Q7: BC858C-7-F, DB_Transistors:SOT-23-3_B-E-C, F.Cu at (216.1, 75.1)
- added Q8: 600V 1.25A, Package_TO_SOT_SMD:SOT-223-3_TabPin2, F.Cu at (236.4, 138.2)
- added Q9: BC858C-7-F, DB_Transistors:SOT-23-3_B-E-C, F.Cu at (216.1, 79.7)
- added R1: 220, DB_SMD_Resistors:R_0603_1608Metric_Pad0.98x0.95mm_HandSolder, F.Cu at (142.0, 63.7)
- added R10: 10K, DB_SMD_Resistors:R_0603_1608Metric_Pad0.98x0.95mm_HandSolder, F.Cu at (133.8, 68.0)
- added R11: 220, DB_SMD_Resistors:R_0603_1608Metric_Pad0.98x0.95mm_HandSolder, F.Cu at (163.9, 63.7)
- added R12: 1K, DB_SMD_Resistors:R_0603_1608Metric_Pad0.98x0.95mm_HandSolder, F.Cu at (210.2, 45.0)
- added R13: 330, DB_SMD_Resistors:R_0603_1608Metric_Pad0.98x0.95mm_HandSolder, F.Cu at (210.2, 47.5)
- added R14: 1K, DB_SMD_Resistors:R_0603_1608Metric_Pad0.98x0.95mm_HandSolder, F.Cu at (210.2, 50.1)
- added R15: 9.1K, DB_SMD_Resistors:R_0603_1608Metric_Pad0.98x0.95mm_HandSolder, F.Cu at (210.2, 52.6)
- added R16: DNP, DB_SMD_Resistors:R_0603_1608Metric_Pad0.98x0.95mm_HandSolder_DNP, F.Cu at (210.2, 55.1)
- added R17: 12K, DB_SMD_Resistors:R_0603_1608Metric_Pad0.98x0.95mm_HandSolder, F.Cu at (141.1, 71.6)
- added R18: 220, DB_SMD_Resistors:R_0603_1608Metric_Pad0.98x0.95mm_HandSolder, F.Cu at (156.6, 63.7)
- added R19: 2.61K, DB_SMD_Resistors:R_0603_1608Metric_Pad0.98x0.95mm_HandSolder, F.Cu at (214.5, 35.0)
- added R2: 330, DB_SMD_Resistors:R_0603_1608Metric_Pad0.98x0.95mm_HandSolder, F.Cu at (205.8, 47.5)
- added R20: DNP, DB_SMD_Resistors:R_0603_1608Metric_Pad0.98x0.95mm_HandSolder_DNP, F.Cu at (214.5, 37.5)
- added R21: 12K, DB_SMD_Resistors:R_0603_1608Metric_Pad0.98x0.95mm_HandSolder, F.Cu at (133.8, 71.6)
- added R22: 330, DB_SMD_Resistors:R_0603_1608Metric_Pad0.98x0.95mm_HandSolder, F.Cu at (214.5, 42.5)
- added R23: 1K, DB_SMD_Resistors:R_0603_1608Metric_Pad0.98x0.95mm_HandSolder, F.Cu at (214.5, 45.0)
- added R24: 1K, DB_SMD_Resistors:R_0603_1608Metric_Pad0.98x0.95mm_HandSolder, F.Cu at (214.5, 47.5)
- added R25: 10K, DB_SMD_Resistors:R_0603_1608Metric_Pad0.98x0.95mm_HandSolder, F.Cu at (214.5, 50.1)
- added R26: 10K, DB_SMD_Resistors:R_0603_1608Metric_Pad0.98x0.95mm_HandSolder, F.Cu at (163.1, 68.0)
- added R27: 10K, DB_SMD_Resistors:R_0603_1608Metric_Pad0.98x0.95mm_HandSolder, F.Cu at (214.5, 55.1)
- added R28: 10K, DB_SMD_Resistors:R_0603_1608Metric_Pad0.98x0.95mm_HandSolder, F.Cu at (155.8, 68.0)
- added R29: 1K, DB_SMD_Resistors:R_0603_1608Metric_Pad0.98x0.95mm_HandSolder, F.Cu at (218.9, 32.5)
- added R3: 220, DB_SMD_Resistors:R_0603_1608Metric_Pad0.98x0.95mm_HandSolder, F.Cu at (134.7, 63.7)
- added R30: 9.1K, DB_SMD_Resistors:R_0603_1608Metric_Pad0.98x0.95mm_HandSolder, F.Cu at (218.9, 35.0)
- added R31: DNP, DB_SMD_Resistors:R_0603_1608Metric_Pad0.98x0.95mm_HandSolder_DNP, F.Cu at (218.9, 37.5)
- added R32: 12K, DB_SMD_Resistors:R_0603_1608Metric_Pad0.98x0.95mm_HandSolder, F.Cu at (163.1, 71.6)
- added R33: 1K, DB_SMD_Resistors:R_0603_1608Metric_Pad0.98x0.95mm_HandSolder, F.Cu at (218.9, 42.5)
- added R34: 2.61K, DB_SMD_Resistors:R_0603_1608Metric_Pad0.98x0.95mm_HandSolder, F.Cu at (218.9, 45.0)
- added R35: DNP, DB_SMD_Resistors:R_0603_1608Metric_Pad0.98x0.95mm_HandSolder_DNP, F.Cu at (218.9, 47.5)
- added R36: 12K, DB_SMD_Resistors:R_0603_1608Metric_Pad0.98x0.95mm_HandSolder, F.Cu at (155.8, 71.6)
- added R37: 220, DB_SMD_Resistors:R_0603_1608Metric_Pad0.98x0.95mm_HandSolder, F.Cu at (149.3, 63.7)
- added R38: 330, DB_SMD_Resistors:R_0603_1608Metric_Pad0.98x0.95mm_HandSolder, F.Cu at (218.9, 55.1)
- added R39: 1K, DB_SMD_Resistors:R_0603_1608Metric_Pad0.98x0.95mm_HandSolder, F.Cu at (218.9, 57.6)
- added R4: 330, DB_SMD_Resistors:R_0603_1608Metric_Pad0.98x0.95mm_HandSolder, F.Cu at (205.8, 52.6)
- added R40: 10K, DB_SMD_Resistors:R_0603_1608Metric_Pad0.98x0.95mm_HandSolder, F.Cu at (223.2, 32.5)
- added R41: 10K, DB_SMD_Resistors:R_0603_1608Metric_Pad0.98x0.95mm_HandSolder, F.Cu at (148.4, 68.0)
- added R42: 1K, DB_SMD_Resistors:R_0603_1608Metric_Pad0.98x0.95mm_HandSolder, F.Cu at (223.2, 37.5)
- added R43: 1.74K, DB_SMD_Resistors:R_0603_1608Metric_Pad0.98x0.95mm_HandSolder, F.Cu at (223.2, 40.0)
- added R44: DNP, DB_SMD_Resistors:R_0603_1608Metric_Pad0.98x0.95mm_HandSolder_DNP, F.Cu at (223.2, 42.5)
- added R45: 12K, DB_SMD_Resistors:R_0603_1608Metric_Pad0.98x0.95mm_HandSolder, F.Cu at (148.4, 71.6)
- added R5: 1K, DB_SMD_Resistors:R_0603_1608Metric_Pad0.98x0.95mm_HandSolder, F.Cu at (205.8, 55.1)
- added R6: 1K, DB_SMD_Resistors:R_0603_1608Metric_Pad0.98x0.95mm_HandSolder, F.Cu at (205.8, 57.6)
- added R7: 10K, DB_SMD_Resistors:R_0603_1608Metric_Pad0.98x0.95mm_HandSolder, F.Cu at (210.2, 32.5)
- added R8: 10K, DB_SMD_Resistors:R_0603_1608Metric_Pad0.98x0.95mm_HandSolder, F.Cu at (141.1, 68.0)
- added R9: 10K, DB_SMD_Resistors:R_0603_1608Metric_Pad0.98x0.95mm_HandSolder, F.Cu at (210.2, 37.5)
- added TP1: TestPoint, DB_TH_Test_Point:TestPoint_Keystone_5005_Compact_Red, F.Cu at (167.1, 68.0)
- added TP2: TestPoint, DB_TH_Test_Point:TestPoint_Keystone_5005_Compact_Red, F.Cu at (159.8, 68.0)
- added TP3: TestPoint, DB_TH_Test_Point:TestPoint_Keystone_5005_Compact_Red, F.Cu at (145.1, 68.0)
- added TP4: TestPoint, DB_TH_Test_Point:TestPoint_Keystone_5005_Compact_Red, F.Cu at (137.8, 68.0)
- added TP5: TestPoint, DB_TH_Test_Point:TestPoint_Keystone_5005_Compact_Red, F.Cu at (152.5, 68.0)
- added TP6: TestPoint, DB_TH_Test_Point:TestPoint_Keystone_5006_Compact_Black, F.Cu at (173.5, 63.5)
- added U10: TL431DBZ-SOT-23, Package_TO_SOT_SMD:SOT-23, F.Cu at (152.5, 74.1)
- added U6: TL431DBZ-SOT-23, Package_TO_SOT_SMD:SOT-23, F.Cu at (167.1, 74.1)
- added U7: TL431DBZ-SOT-23, Package_TO_SOT_SMD:SOT-23, F.Cu at (211.0, 65.9)
- added U8: TL431DBZ-SOT-23, Package_TO_SOT_SMD:SOT-23, F.Cu at (159.8, 74.1)
- added U9: TL431DBZ-SOT-23, Package_TO_SOT_SMD:SOT-23, F.Cu at (211.0, 75.1)
- FH1: value 3.5A -> 6.3A
- FH3: value 6.3A -> 0.08A
- FH5: value 0.1A -> 3.5A
- Q1, Q2, Q5: value 600V, 8A -> BC858C-7-F; footprint Package_TO_SOT_SMD:TO-252-2 -> DB_Transistors:SOT-23-3_B-E-C
- Q3, Q4: value 600V, 8A -> 600V 1.25A; footprint Package_TO_SOT_SMD:TO-252-2 -> Package_TO_SOT_SMD:SOT-223-3_TabPin2
- moved U4 119.3 mm to (137.9, 74.1), turned to -90 degrees
- moved U2 111.7 mm to (145.2, 74.1), turned to -90 degrees
- moved FH1 78.8 mm to (225.4, 120.7)
- moved FH2 78.8 mm to (225.4, 127.2)
- moved FH3 78.8 mm to (225.4, 133.8)
- moved FH4 78.8 mm to (225.4, 140.4)
- moved FH5 78.8 mm to (225.4, 147.0)
- moved Q4 61.6 mm to (236.4, 129.9)
- moved Q3 61.5 mm to (236.4, 121.6)
- moved U1 51.3 mm to (206.1, 61.2)
- moved U3 51.3 mm to (206.1, 70.5)
- moved U5 51.3 mm to (206.1, 79.7)
- moved Q1 21.5 mm to (216.1, 61.2)
- moved Q2 18.8 mm to (216.1, 65.9)
- moved Q5 14.5 mm to (216.1, 70.5)
Connections:
- FH1 pad 1: unconnected-(FH1-Pad1) -> +5V
- FH1 pad 2: unconnected-(FH1-Pad2) -> +5V_Fused
- FH2 pad 1: unconnected-(FH2-Pad1) -> +12V
- FH2 pad 2: unconnected-(FH2-Pad2) -> +12V_Fused
- FH3 pad 1: unconnected-(FH3-Pad1) -> -5V
- FH3 pad 2: unconnected-(FH3-Pad2) -> -5V_Fused
- FH4 pad 1: unconnected-(FH4-Pad1) -> -12V
- FH4 pad 2: unconnected-(FH4-Pad2) -> -12V_Fused
- FH5 pad 1: unconnected-(FH5-Pad1) -> +15V
- FH5 pad 2: unconnected-(FH5-Pad2) -> +15V_Fused
- MH1 pad 1: unconnected-(MH1-Pad1) -> GND
- MH2 pad 1: unconnected-(MH2-Pad1) -> GND
- Q3 pad 1: unconnected-(Q3-K-Pad1) -> -5V_Fused
- Q3 pad 2: unconnected-(Q3-A-Pad2) -> GND
- Q3 pad 3: unconnected-(Q3-G-Pad3) -> Net-(Q1-B)
- Q4 pad 1: unconnected-(Q4-K-Pad1) -> -12V_Fused
- Q4 pad 2: unconnected-(Q4-A-Pad2) -> GND
- Q4 pad 3: unconnected-(Q4-G-Pad3) -> Net-(Q2-E)
- U1 pad 1: unconnected-(U1-K-Pad1) -> Net-(U1-K)
- U1 pad 2: unconnected-(U1-REF-Pad2) -> Net-(U1-REF)
- U1 pad 3: unconnected-(U1-A-Pad3) -> -5V_Fused
- U2 pad 1: unconnected-(U2-K-Pad1) -> Net-(LD3-K)
- U2 pad 2: unconnected-(U2-REF-Pad2) -> Net-(U6-REF)
- U2 pad 3: unconnected-(U2-A-Pad3) -> GND
- U3 pad 1: unconnected-(U3-K-Pad1) -> Net-(U3-K)
- U3 pad 2: unconnected-(U3-REF-Pad2) -> Net-(U3-REF)
- U3 pad 3: unconnected-(U3-A-Pad3) -> -12V_Fused
- U4 pad 1: unconnected-(U4-K-Pad1) -> Net-(LD3-K)
- U4 pad 2: unconnected-(U4-REF-Pad2) -> Net-(U6-REF)
- U4 pad 3: unconnected-(U4-A-Pad3) -> GND
- U5 pad 1: unconnected-(U5-K-Pad1) -> Net-(U5-K)
- U5 pad 2: unconnected-(U5-REF-Pad2) -> Net-(U5-REF)
- U5 pad 3: unconnected-(U5-A-Pad3) -> GND
Routing:
- net Net-(LD3-K): track 0.00 -> 52.3 mm
- net +5V_Fused: track 0.00 -> 40.8 mm
- net Net-(U6-REF): track 0.00 -> 29.4 mm
- net GND: track 0.00 -> 28.4 mm, vias 0 -> 5
- net Net-(LD3-A): track 0.00 -> 8.01 mm
- added copper zone on B.Cu, net GND
Other:
- copper layers 2 -> 4
- board text added: "+12V PWR GD"
- board text added: "+15V PWR GD"
- board text added: "+5V PWR GD"
- board text added: "-12V PWR GD"
- board text added: "-5V PWR GD"
- board text added: "GND"

Commit message: First draft of layout
Parts:
- R18, R3: value 220 -> 1.5K
- R21, R36: value 12K -> 2.94K
- R37: value 220 -> 2.2K
- R45: value 12K -> 2.2K
- moved Q3 130.0 mm to (116.1, 72.4), turned to -90 degrees
- moved R33 127.4 mm to (124.7, 128.4)
- moved Q4 122.5 mm to (119.9, 92.4), turned to 90 degrees
- moved C4 120.4 mm to (121.0, 125.5), turned to 90 degrees
- moved R24 119.6 mm to (121.5, 122.7), turned to 180 degrees
- moved R22 119.1 mm to (124.7, 120.8), turned to 180 degrees
- moved R34 118.9 mm to (122.7, 114.9)
- moved R40 117.6 mm to (155.4, 128.5)
- moved R35 116.5 mm to (122.7, 113.3)
- moved FH3 115.9 mm to (125.8, 74.5)
- moved R7 115.7 mm to (106.0, 82.9), turned to -90 degrees
- moved R27 112.7 mm to (120.9, 117.9), turned to 90 degrees
- moved R20 109.8 mm to (114.5, 82.9), turned to -90 degrees
- moved R19 109.4 mm to (116.2, 82.9), turned to -90 degrees
- moved FH4 108.1 mm to (124.0, 103.3), turned to 180 degrees
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Connections:
- J1 pad 1: -12V -> +15V
- J1 pad 2: -5V -> +12V
- J1 pad 3: GND -> -12V
- J1 pad 5: +15V -> -5V
- J1 pad 6: +12V -> GND
- J2 pad 2: -5V_Fused -> +12V_Fused
- J2 pad 3: GND -> +15V_Fused
- J2 pad 5: +5V_Fused -> -5V_Fused
- J2 pad 6: +15V_Fused -> unconnected-(J2-Pin_6-Pad6)
- J2 pad 7: +12V_Fused -> +5V_Fused
- LD1 pad 1: Net-(LD3-K) -> Net-(LD1-K)
- LD1 pad 2: Net-(LD3-A) -> Net-(LD1-A)
- LD2 pad 1: Net-(LD3-K) -> Net-(LD2-K)
- LD2 pad 2: Net-(LD3-A) -> Net-(LD2-A)
- LD4 pad 1: Net-(LD3-K) -> Net-(LD4-K)
- LD4 pad 2: Net-(LD3-A) -> Net-(LD4-A)
- LD5 pad 1: Net-(LD3-K) -> Net-(LD5-K)
- LD5 pad 2: Net-(LD3-A) -> Net-(LD5-A)
- R1 pad 1: +5V_Fused -> GND
- R1 pad 2: Net-(LD3-A) -> Net-(LD1-A)
- R10 pad 1: +5V_Fused -> GND
- R10 pad 2: Net-(U6-REF) -> Net-(U4-REF)
- R17 pad 1: Net-(U6-REF) -> Net-(U2-REF)
- R17 pad 2: GND -> -5V_Fused
- R18 pad 1: +5V_Fused -> +12V_Fused
- R18 pad 2: Net-(LD3-A) -> Net-(LD4-A)
- R21 pad 1: Net-(U6-REF) -> Net-(U4-REF)
- R21 pad 2: GND -> -12V_Fused
- R28 pad 1: +5V_Fused -> +12V_Fused
- R28 pad 2: Net-(U6-REF) -> Net-(U8-REF)
- R3 pad 1: +5V_Fused -> GND
- R3 pad 2: Net-(LD3-A) -> Net-(LD2-A)
- R36 pad 1: Net-(U6-REF) -> Net-(U8-REF)
- R37 pad 1: +5V_Fused -> +15V_Fused
- R37 pad 2: Net-(LD3-A) -> Net-(LD5-A)
- R41 pad 1: +5V_Fused -> +15V_Fused
- R41 pad 2: Net-(U6-REF) -> Net-(U10-REF)
- R45 pad 1: Net-(U6-REF) -> Net-(U10-REF)
- R8 pad 1: +5V_Fused -> GND
- R8 pad 2: Net-(U6-REF) -> Net-(U2-REF)
- TP2 pad 1: +5V_Fused -> +12V_Fused
- TP3 pad 1: +5V_Fused -> -5V_Fused
- TP4 pad 1: +5V_Fused -> -12V_Fused
- TP5 pad 1: +5V_Fused -> +15V_Fused
- U10 pad 1: Net-(LD3-K) -> Net-(LD5-K)
- U10 pad 2: Net-(U6-REF) -> Net-(U10-REF)
- U2 pad 1: Net-(LD3-K) -> Net-(LD1-K)
- U2 pad 2: Net-(U6-REF) -> Net-(U2-REF)
- U2 pad 3: GND -> -5V_Fused
- U4 pad 1: Net-(LD3-K) -> Net-(LD2-K)
- U4 pad 2: Net-(U6-REF) -> Net-(U4-REF)
- U4 pad 3: GND -> -12V_Fused
- U8 pad 1: Net-(LD3-K) -> Net-(LD4-K)
- U8 pad 2: Net-(U6-REF) -> Net-(U8-REF)
Routing:
- net -5V_Fused: track 0.00 -> 108.1 mm
- net -12V_Fused: track 0.00 -> 91.2 mm, vias 0 -> 3
- net +12V_Fused: track 0.00 -> 68.2 mm, vias 0 -> 3
- net +15V_Fused: track 0.00 -> 45.3 mm
- net Net-(LD3-K): track 52.3 -> 10.5 mm
- net -5V: track 0.00 -> 36.0 mm
- net Net-(U6-REF): track 29.4 -> 5.89 mm
- net GND: track 28.4 -> 45.2 mm
- net Net-(U5-K): track 0.00 -> 14.9 mm
- net Net-(U3-K): track 0.00 -> 13.9 mm
- net Net-(U9-K): track 0.00 -> 13.1 mm
- net Net-(Q4-G): track 0.00 -> 11.6 mm
- net Net-(LD1-K): track 0.00 -> 10.5 mm
- net Net-(LD5-K): track 0.00 -> 10.5 mm
- net Net-(LD4-K): track 0.00 -> 10.5 mm
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Other:
- copper layers 4 -> 2
- board text added: "+12V Fuse"
- board text added: "+15V Fuse"
- board text added: "+5V Fuse"
- board text added: "-12V Fuse"
- board text added: "-5V Fuse"
- board text added: "0.08A"
- board text added: "0.1A"
- board text added: "0.4A"
- board text added: "3.5A"
- board text added: "6.3A"

Commit message: Ready to send to production
Parts:
- added GL1: ~, DB_Logo_Footprints:Myscion_Dynamics_Main, F.Cu at (172.1, 130.0)
- moved R4 15.0 mm to (119.3, 97.2)
- moved R6 14.3 mm to (119.5, 94.5)
- moved Q2 14.1 mm to (116.0, 97.4)
- moved C2 14.1 mm to (116.0, 94.5)
- moved R14 13.8 mm to (118.2, 100.6), turned to 180 degrees
- moved Q4 13.4 mm to (116.1, 105.2), turned to 180 degrees
- moved U3 12.9 mm to (123.4, 95.0)
- moved R9 12.4 mm to (123.4, 91.1)
- moved Q3 9.92 mm to (125.5, 69.2)
- moved C1 9.92 mm to (119.8, 75.1)
- moved Q1 9.92 mm to (119.8, 72.0)
- moved R12 9.92 mm to (120.8, 67.8)
- moved R15 9.92 mm to (119.3, 82.4)
- moved R16 9.92 mm to (119.3, 83.9)
- moved R2 9.92 mm to (118.2, 76.7)
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Connections:
- J2 pad 6: unconnected-(J2-Pin_6-Pad6) -> GND
Routing:
- net +15V_Fused: track 45.3 -> 93.0 mm, vias 0 -> 8
- net +12V_Fused: track 68.2 -> 113.9 mm, vias 3 -> 6
- net GND: track 45.2 -> 87.2 mm, vias 5 -> 73
- net +5V_Fused: track 43.0 -> 73.9 mm, vias 0 -> 3
- net -12V_Fused: track 91.2 -> 113.2 mm, vias 3 -> 5
- net -5V: track 36.0 -> 26.7 mm
- net Net-(Q4-G): track 11.6 -> 5.65 mm
- net +12V: track 9.22 -> 14.1 mm
- net -12V: track 8.97 -> 12.8 mm
- net +5V: track 6.66 -> 9.45 mm
- net Net-(U5-K): track 14.9 -> 17.5 mm
- net -5V_Fused: track 108.1 -> 106.0 mm
- net +15V: track 7.17 -> 9.22 mm
- net Net-(U3-K): track 13.9 -> 12.9 mm, vias 0 -> 2
- net Net-(U3-REF): track 5.96 -> 7.00 mm
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- added copper zone on F.Cu, net GND
Other:
- board text added: "HP9815 OVP BOARD"
- board text added: "If the proper fuses can not be found any fast 2512 fuse can be used instead."
- board text added: "JLCJLCJLCJLC"
- board text added: "Replacement Fuses +15V 3.5A: 45303.5, 45103.5, 44803.5 +12V 0.4A: 453.4, 451.4, 448.4 +5V 6.3A: 45306.3, 45106.3, 44806.3 -5V 0.08A: 453.08, 451.08, 448.08 -12V 0.1A: 453.1, 451.1, 448.1"
- board text added: "Rev - 08/2025"
- board text added: "This board intercepts all the power rails in the HP9815a and probvides over voltage protection. If voltage rises too high crow bar circuits will trip and blow the fuse."

Commit message: Sent PCB out to fab
Parts:
- added GL2: ~, Symbol:OSHW-Logo_11.4x12mm_SilkScreen, F.Cu at (107.8, 127.3)
Routing:
- net -12V_Fused: track 113.2 -> 114.3 mm
- net GND: vias 73 -> 78
Other:
- board text added: "This board intercepts all the power rails in the HP9815 and provides over voltage protection. If voltage rises too high crow bar circuits will trip and blow the fuse."
- board text added: "To view the source files please visit my github: https://github.com/Myscion-Dynamics/HP9815_OVP"
- board text removed: "This board intercepts all the power rails in the HP9815a and probvides over voltage protection. If voltage rises too high crow bar circuits will trip and blow the fuse."
