File: HP9815_OVP_Schematic/HP9815_OVP/HP9815_OVP.kicad_sch (KiCad schematic)
At the start: 19 parts, among them Q1 600V, 8A, Q2 600V, 8A, Q3 600V, 8A, Q4 600V, 8A, Q5 600V, 8A, U1 TL431DBZ-SOT-23, U2 TL431DBZ-SOT-23, U3 TL431DBZ-SOT-23, U4 TL431DBZ-SOT-23, U5 TL431DBZ-SOT-23

Commit message: Simulated started and outline done
Parts:
- removed MH3, MH4: 3mm, DB_Mounting_Holes:MountingHole_3.2mm_M3_Pad, symbol DB:Mounting_Holes/3mm-plated-hole
- added J1: IPBT-103-H1-T-D-K, DB_Connector_Samtec:SAMTEC_IPBT-103-H1-T-D-K, symbol DB:Connector_Samtec/SAM9554-ND
- added J2: IPBT-104-H1-T-D-K, DB_Connector_Samtec:SAMTEC_IPBT-104-H1-T-D-K, symbol DB:Connector_Samtec/SAM9558-ND
Other:
- note added: "Mating Conn: IPBD-03-D-K 16-20AWG Crimp: CC69L-1620-01-T-SP 20-24 AWG Crimp: CC69L-2024-01-T-SP"
- note added: "Mating Conn: IPBD-04-D-K 16-20AWG Crimp: CC69L-1620-01-T-SP 20-24 AWG Crimp: CC69L-2024-01-T-SP"
Changed lines of the file:
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@@
+		)
+	)
+	(text "Mating Conn: IPBD-04-D-K\n16-20AWG Crimp: CC69L-1620-01-T-SP\n20-24 AWG Crimp: CC69L-2024-01-T-SP"
+		(exclude_from_sim no)
+		(at 190.5 147.32 0)
+		(effects
+			(font
+				(size 1.27 1.27)
+			)
 		)
 	)
@@
 		(exclude_from_sim no)
 		(at 175.26 35.56 0)
+		(effects
+			(font
+				(size 1.27 1.27)
+			)
+		)
+	)
+	(text "Mating Conn: IPBD-03-D-K\n16-20AWG Crimp: CC69L-1620-01-T-SP\n20-24 AWG Crimp: CC69L-2024-01-T-SP"
+		(exclude_from_sim no)
+		(at 142.24 147.32 0)
 		(effects
 			(font
@@
 	)
 	(symbol
+		(lib_id "DB:Connector_Samtec/SAM9558-ND")
+		(at 177.8 135.89 0)
+		(unit 1)
+		(exclude_from_sim no)
+		(in_bom yes)
+		(on_board yes)
+		(dnp no)
+		(fields_autoplaced yes)
+		(property "Reference" "J2"
+			(at 177.673 125.73 0)
+			(effects
+				(font
+					(size 1.27 1.27)
+				)
+			)
+		)
+		(property "Value" "IPBT-104-H1-T-D-K"
+			(at 178.562 142.748 0)
+			(effects
+				(font
+					(size 1.27 1.27)
+				)
+				(hide yes)
+			)
+		)
+		(property "Footprint" "DB_Connector_Samtec:SAMTEC_IPBT-104-H1-T-D-K"
+			(at 177.8 135.89 0)
+			(effects
+				(font
+					(size 1.27 1.27)
+				)
+				(hide yes)
+			)
+		)
+		(property "Datasheet" "~"
+			(at 177.8 135.89 0)
+			(effects
+				(font
+					(size 1.27 1.27)
+				)
+				(hide yes)
+			)
+		)
+		(property "Description" "Connector Header Through Hole 8 position 0.165\" (4.20mm)"
+			(at 182.88 130.81 0)
+			(effects
+				(font
+					(size 1.27 1.27)
+				)
+				(hide yes)
+			)
+		)
+		(property "MPN" "IPBT-104-H1-T-D-K"
+			(at 177.673 128.27 0)
+			(effects
+				(font
+					(size 1.27 1.27)
+				)
+			)
+		)
+		(property "Positions" "8"
+			(at 177.8 135.89 0)
+			(effects
+				(font
+					(size 1.27 1.27)
+				)
+				(hide yes)
+			)
+		)
+		(property "Disc" "Connector Header Through Hole 8 position 0.165\" (4.20mm)"
+			(at 177.8 135.89 0)
+			(effects
+				(font
+					(size 1.27 1.27)
+				)
+				(hide yes)
+			)
+		)
+		(property "Manufacture" "Samtec Inc."
+			(at 177.8 135.89 0)
+			(effects
+				(font
+					(size 1.27 1.27)
+				)
+				(hide yes)
+			)
+		)
+		(property "Current" "9.3A"
+			(at 177.8 135.89 0)
+			(effects
+				(font
+					(size 1.27 1.27)
+				)
+				(hide yes)
+			)
+		)
+		(property "Voltage" "400VAC, 565VDC"
+			(at 177.8 135.89 0)
+			(effects
+				(font
+					(size 1.27 1.27)
+				)
+				(hide yes)
+			)
+		)
+		(pin "8"
+		)
+		(pin "6"
+		)
+		(pin "5"
+		)
+		(pin "7"
+		)
+		(pin "4"
+		)
+		(pin "1"
+		)
+		(pin "3"
+		)
+		(pin "2"
+		)
+		(instances
+			(project ""
+				(path "/ba2b9114-e1a5-46b3-b25b-16fdae1043bd"
+					(reference "J2")
+					(unit 1)
+				)
+			)
+		)
+	)
+	(symbol
 		(lib_id "DB:Fuse_in_Holder/0.1A Fast")
 		(at 171.45 73.66 0)
@@
 	)
 	(symbol
-		(lib_id "DB:Mounting_Holes/3mm-plated-hole")
-		(at 67.31 140.97 0)
+		(lib_id "DB:Connector_Samtec/SAM9554-ND")
+		(at 149.86 134.62 0)
 		(unit 1)
 		(exclude_from_sim no)
@@
 		(dnp no)
 		(fields_autoplaced yes)
-		(property "Reference" "MH4"
-			(at 69.85 138.4299 0)
-			(effects
-				(font
-					(size 1.27 1.27)
-				)
-				(justify left)
-			)
-		)
-		(property "Value" "3mm"
-			(at 69.85 140.9699 0)
-			(effects
-				(font
-					(size 1.27 1.27)
-				)
-				(justify left)
-			)
-		)
-		(property "Footprint" "DB_Mounting_Holes:MountingHole_3.2mm_M3_Pad"
-			(at 67.31 140.97 0)
+		(property "Reference" "J1"
+			(at 149.7965 125.73 0)
+			(effects
+				(font
+					(size 1.27 1.27)
+				)
+			)
+		)
+		(property "Value" "IPBT-103-H1-T-D-K"
+			(at 150.622 140.208 0)
+			(effects
+				(font
+					(size 1.27 1.27)
+				)
+				(hide yes)
+			)
+		)
+		(property "Footprint" "DB_Connector_Samtec:SAMTEC_IPBT-103-H1-T-D-K"
+			(at 149.86 134.62 0)
 			(effects
 				(font
@@
 		)
 		(property "Datasheet" "~"
-			(at 67.31 140.97 0)
-			(effects
-				(font
-					(size 1.27 1.27)
-				)
-				(hide yes)
-			)
-		)
-		(property "Description" "3mm plated hole"
-			(at 67.31 140.97 0)
-			(effects
-				(font
-					(size 1.27 1.27)
-				)
-				(hide yes)
-			)
-		)
-		(property "Type" "Plated"
-			(at 67.31 140.97 0)
-			(effects
-				(font
-					(size 1.27 1.27)
-				)
-				(hide yes)
-			)
+			(at 149.86 134.62 0)
+			(effects
+				(font
+					(size 1.27 1.27)
+				)
+				(hide yes)
+			)
+		)
+		(property "Description" "Connector Header Through Hole 6 position 0.165\" (4.20mm)"
+			(at 154.94 129.54 0)
+			(effects
+				(font
+					(size 1.27 1.27)
+				)
+				(hide yes)
+			)
+		)
+		(property "MPN" "IPBT-103-H1-T-D-K"
+			(at 149.7965 128.27 0)
+			(effects
+				(font
+					(size 1.27 1.27)
+				)
+			)
+		)
+		(property "Positions" "6"
+			(at 149.86 134.62 0)
+			(effects
+				(font
+					(size 1.27 1.27)
+				)
+				(hide yes)
+			)
+		)
+		(property "Disc" "Connector Header Through Hole 6 position 0.165\" (4.20mm)"
+			(at 149.86 134.62 0)
+			(effects
+				(font
+					(size 1.27 1.27)
+				)
+				(hide yes)
+			)
+		)
+		(property "Manufacture" "Samtec Inc."
+			(at 149.86 134.62 0)
+			(effects
+				(font
+					(size 1.27 1.27)
+				)
+				(hide yes)
+			)
+		)
+		(property "Current" "9.3A"
+			(at 149.86 134.62 0)
+			(effects
+				(font
+					(size 1.27 1.27)
+				)
+				(hide yes)
+			)
+		)
+		(property "Voltage" "400VAC, 565VDC"
+			(at 149.86 134.62 0)
+			(effects
+				(font
+					(size 1.27 1.27)
+				)
+				(hide yes)
+			)
+		)
+		(pin "4"
+		)
+		(pin "5"
 		)
 		(pin "1"
 		)
+		(pin "2"
+		)
+		(pin "6"
+		)
+		(pin "3"
+		)
 		(instances
-			(project "HP9815_OVP"
+			(project ""
 				(path "/ba2b9114-e1a5-46b3-b25b-16fdae1043bd"
-					(reference "MH4")
+					(reference "J1")
 					(unit 1)
 				)
@@
 					(unit 1)
 				)
-			)
-		)
-	)
-	(symbol
-		(lib_id "DB:Mounting_Holes/3mm-plated-hole")
-		(at 63.5 156.21 0)
-		(unit 1)
-		(exclude_from_sim no)
-		(in_bom yes)
-		(on_board yes)
-		(dnp no)
-		(fields_autoplaced yes)
-		(property "Reference" "MH3"
-			(at 66.04 153.6699 0)
-			(effects
-				(font
-					(size 1.27 1.27)
-				)
-				(justify left)
-			)
-		)
-		(property "Value" "3mm"
-			(at 66.04 156.2099 0)
-			(effects
-				(font
-					(size 1.27 1.27)
-				)
-				(justify left)
-			)
-		)
-		(property "Footprint" "DB_Mounting_Holes:MountingHole_3.2mm_M3_Pad"
-			(at 63.5 156.21 0)
-			(effects
-				(font
-					(size 1.27 1.27)
-				)
-				(hide yes)
-			)
-		)
-		(property "Datasheet" "~"
-			(at 63.5 156.21 0)
-			(effects
-				(font
-					(size 1.27 1.27)
-				)
-				(hide yes)
-			)
-		)
-		(property "Description" "3mm plated hole"
-			(at 63.5 156.21 0)
-			(effects
-				(font
-					(size 1.27 1.27)
-				)
-				(hide yes)
-			)
-		)
-		(property "Type" "Plated"
-			(at 63.5 156.21 0)
-			(effects
-				(font
-					(size 1.27 1.27)
-				)
-				(hide yes)
-			)
-		)
-		(pin "1"
-		)
-		(instances
-			(project "HP9815_OVP"
-				(path "/ba2b9114-e1a5-46b3-b25b-16fdae1043bd"
-					(reference "MH3")
-					(unit 1)
-				)

Commit message: Commit before relinking ref des
Parts:
- removed FH5: 0.1A, DB_Fuse_in_Holder:Fuseholder_Littelfuse_Nano2_154x, symbol DB:Fuse_in_Holder/0.1A Fast
- removed Q1, Q2, Q4, Q5: 600V, 8A, Package_TO_SOT_SMD:TO-252-2, symbol DB:SCR/SCR 600V 8A DPAK
- removed U5: TL431DBZ-SOT-23, Package_TO_SOT_SMD:SOT-23, symbol DB:Reference_Voltage_Source/296-17329-1-ND
- added C1, C2, C3, C4, C5: 10nF, DB_SMD_Capacitors:C_0603_1608Metric_Pad1.08x0.95mm_HandSolder, symbol DB:Ceramic_0603_X7R_50V/CAP CER 10000PF 50V X7R 0603
- added FH3: 0.08A, DB_Fuse_in_Holder:Fuseholder_Littelfuse_Nano2_154x, symbol DB:Fuse_in_Holder/0.08A Fast
- added LD1, LD2, LD3, LD4, LD5: Green, DB_SMD_LED:LED_0603_1608Metric_Green_Cath_Dot, symbol DB:LED_SMD_0603/LED GREEN DIFFUSED 0603 SMD
- added Q1, Q2, Q5, Q7, Q9: BC858C-7-F, DB_Transistors:SOT-23-3_B-E-C, symbol DB:Transistor_SMD_PNP/TRANS PNP 30V 0.1A SOT-23-3
- added Q10: 600V, 8A, Package_TO_SOT_SMD:TO-252-2, symbol DB:SCR/SCR 600V 8A DPAK
- added Q3, Q4, Q8: 600V 1.25A, Package_TO_SOT_SMD:SOT-223-3_TabPin2, symbol DB:SCR/SCR 600 V 1.25 A Sensitive Gate Surface Mount SOT-223
- added R1, R11: 220, DB_SMD_Resistors:R_0603_1608Metric_Pad0.98x0.95mm_HandSolder, symbol DB:Resistor_SMD_0603/RES 220 OHM 1% 1/10W SMD
- added R10, R25, R26, R27, R28, R40, R41, R7, R8, R9: 10K, DB_SMD_Resistors:R_0603_1608Metric_Pad0.98x0.95mm_HandSolder, symbol DB:Resistor_SMD_0603/RES 10K OHM 1% 1/10W SMD
- added R12, R14, R23, R24, R29, R33, R39, R42, R5, R6: 1K, DB_SMD_Resistors:R_0603_1608Metric_Pad0.98x0.95mm_HandSolder, symbol DB:Resistor_SMD_0603/RES 1K OHM 1% 1/10W SMD
- added R13, R2, R22, R38, R4: 330, DB_SMD_Resistors:R_0603_1608Metric_Pad0.98x0.95mm_HandSolder, symbol DB:Resistor_SMD_0603/RES 330 OHM 1% 1/10W SMD
- added R15, R30: 9.1K, DB_SMD_Resistors:R_0603_1608Metric_Pad0.98x0.95mm_HandSolder, symbol DB:Resistor_SMD_0603/RES 9.1K OHM 1% 1/10W SMD
- added R16, R20, R31, R35, R44: DNP, DB_SMD_Resistors:R_0603_1608Metric_Pad0.98x0.95mm_HandSolder_DNP, symbol DB:Resistor_SMD_0603/RES DNP 1/10W SMD
- added R17, R32: 12K, DB_SMD_Resistors:R_0603_1608Metric_Pad0.98x0.95mm_HandSolder, symbol DB:Resistor_SMD_0603/RES 12K OHM 1% 1/10W SMD
- added R18, R3: 1.5K, DB_SMD_Resistors:R_0603_1608Metric_Pad0.98x0.95mm_HandSolder, symbol DB:Resistor_SMD_0603/RES 1.5K OHM 1% 1/10W SMD
- added R19, R34: 2.61K, DB_SMD_Resistors:R_0603_1608Metric_Pad0.98x0.95mm_HandSolder, symbol DB:Resistor_SMD_0603/RES 2.61K OHM 1% 1/10W SMD
- added R21, R36: 2.94K, DB_SMD_Resistors:R_0603_1608Metric_Pad0.98x0.95mm_HandSolder, symbol DB:Resistor_SMD_0603/RES 2.94K OHM 1% 1/10W SMD
- added R37, R45: 2.2K, DB_SMD_Resistors:R_0603_1608Metric_Pad0.98x0.95mm_HandSolder, symbol DB:Resistor_SMD_0603/RES 2.2K OHM 1% 1/10W SMD
- added R43: 1.74K, DB_SMD_Resistors:R_0603_1608Metric_Pad0.98x0.95mm_HandSolder, symbol DB:Resistor_SMD_0603/RES 1.74K OHM 1% 1/10W SMD
- added TP1, TP2, TP3, TP4, TP5: TestPoint, DB_TH_Test_Point:TestPoint_Keystone_5005_Compact_Red, symbol DB:Test_Points_TH/Red_Compact_1.6mmH
- added TP6: TestPoint, DB_TH_Test_Point:TestPoint_Keystone_5006_Compact_Black, symbol DB:Test_Points_TH/Black_Compact_1.6mmH
- added U10, U3, U6, U7, U8, U9: TL431DBZ-SOT-23, Package_TO_SOT_SMD:SOT-23, symbol DB:Reference_Voltage_Source/296-17329-1-ND
- renumbered FH3 to FH1, FH1 to FH5, Q3 to Q6, U3 to U5
Connections:
- net GND: now reaches MH2.1
- net GND: now also J1.3 (Pin_3), J2.3 (Pin_3), J2.4 (Pin_4), J2.8 (Pin_8), MH1.1, Q6.1 (K), U5.3 (A), C1.1, C2.1, Q1.E, Q10.1 (K), Q2.E, Q3.2 (A), Q4.2 (A), Q8.1 (K), R1.1, R10.1, R2.1, R29.1, R3.1, R30.2, R31.2, R32.2, R33.1, R34.2, R35.2, R36.2, R4.1, R42.1, R43.2, R44.2, R45.2, R8.1, TP6.1, U10.3 (A), U6.3 (A), U7.3 (A), U8.3 (A), U9.3 (A)
- net at U2.1 (K): now also LD1.1 (K)
- net at U2.2 (REF): now also R17.1, R8.2
- net -5V_Fused: now reaches U2.3 (A)
- net -5V_Fused: now also J2.2 (Pin_2), U1.3 (A), FH3.2, Q3.1 (K), R12.1, R15.2, R16.2, R17.2, TP3.1
- net -12V_Fused: now reaches J2.1 (Pin_1)
- net -12V_Fused: now also FH4.2, U4.3 (A), Q4.1 (K), R14.1, R19.2, R20.2, R21.2, TP4.1, U3.3 (A)
- net +5V_Fused: now reaches J2.5 (Pin_5)
- net +5V_Fused: now also FH1.2, Q6.2 (A), C3.1, Q5.E, R11.1, R13.1, R26.1, TP1.1
- net +15V_Fused: now reaches J2.6 (Pin_6)
- net +15V_Fused: now also FH5.2, C5.1, Q10.2 (A), Q9.E, R37.1, R38.1, R41.1, TP5.1
- net +12V_Fused: now reaches J2.7 (Pin_7)
- net +12V_Fused: now also FH2.2, C4.1, Q7.E, Q8.2 (A), R18.1, R22.1, R28.1, TP2.1
- net -12V: now reaches FH4.1
- net -12V: now also J1.1 (Pin_1)
- net +12V: now reaches FH2.1
- net +12V: now also J1.6 (Pin_6)
- net at U5.1 (K): now also R13.2, R23.1, R25.1
- net at U5.2 (REF): now also R25.2, R30.1, R31.1
- net at U1.1 (K): now also R2.2, R5.1, R7.1
- net at U1.2 (REF): now also R15.1, R16.1, R7.2
- net +15V: now reaches FH5.1
- net +15V: now also J1.5 (Pin_5)
- net +5V: now reaches FH1.1
- net +5V: now also J1.4 (Pin_4)
- net -5V: now reaches J1.2 (Pin_2)
- net -5V: now also FH3.1
- net at Q6.3 (G): now also Q5.C, R29.2
- net at U4.1 (K): now also LD2.1 (K)
- net at U4.2 (REF): now also R10.2, R21.1
- new net: LD3.2 (A), R11.2
- new net: C2.2, Q2.B, R6.2
- new net: Q2.C, Q4.3 (G), R14.2
- new net: LD2.2 (A), R3.2
- new net: LD3.1 (K), U6.1 (K)
- new net: R26.2, R32.1, U6.2 (REF)
- new net: Q1.C, Q3.3 (G), R12.2
- new net: R38.2, R39.1, R40.1, U9.1 (K)
- new net: R40.2, R43.1, R44.1, U9.2 (REF)
- new net: R41.2, R45.1, U10.2 (REF)
- new net: LD1.2 (A), R1.2
- new net: R4.2, R6.1, R9.1, U3.1 (K)
- new net: R19.1, R20.1, R9.2, U3.2 (REF)
- new net: R22.2, R24.1, R27.1, U7.1 (K)
- new net: R27.2, R34.1, R35.1, U7.2 (REF)
- new net: C1.2, Q1.B, R5.2
- new net: C5.2, Q9.B, R39.2
- new net: C3.2, Q5.B, R23.2
- new net: LD4.2 (A), R18.2
- new net: LD4.1 (K), U8.1 (K)
- new net: R28.2, R36.1, U8.2 (REF)
- new net: Q10.3 (G), Q9.C, R42.2
- new net: LD5.2 (A), R37.2
- new net: Q7.C, Q8.3 (G), R33.2
- new net: LD5.1 (K), U10.1 (K)
- new net: C4.2, Q7.B, R24.2
Other:
- note added: "0.0004 I2t Fusing"
- note added: "0.002 I2t Fusing"
- note added: "0.06 I2t Fusing"
- note added: "2.5 I2t Fusing"
- note added: "60 I2t Fusing"
- note added: "9.2 I2t Fusing"
- note added: "OVP Triggers at -13V"
- note added: "OVP Triggers at -5.85V"
- note added: "OVP Triggers at 13V"
- note added: "OVP Triggers at 17V"
- note added: "OVP Triggers at 5.85V"
- note added: "Power Good Triggers at -11V"
- note added: "Power Good Triggers at -4.6V"
- note added: "Power Good Triggers at 11V"
- note added: "Power Good Triggers at 13.9V"
- note added: "Power Good Triggers at 4.6V"
- moved on the sheet: FH1, FH2, FH5, J1, J2, MH1, Q6, U5

Commit message: First draft of layout
Connections:
- net +12V: now also J1.2 (Pin_2); no longer J1.6 (Pin_6)
- net +12V_Fused: now also J2.2 (Pin_2); no longer J2.7 (Pin_7)
- net +15V: now also J1.1 (Pin_1); no longer J1.5 (Pin_5)
- net +15V_Fused: now also J2.3 (Pin_3); no longer J2.6 (Pin_6)
- net +5V_Fused: now also J2.7 (Pin_7); no longer J2.5 (Pin_5)
- net -12V: now also J1.3 (Pin_3); no longer J1.1 (Pin_1)
- net -5V: now also J1.5 (Pin_5); no longer J1.2 (Pin_2)
- net -5V_Fused: now also J2.5 (Pin_5); no longer J2.2 (Pin_2)
- net GND: now also J1.6 (Pin_6); no longer J1.3 (Pin_3), J2.3 (Pin_3)
Other:
- moved on the sheet: C1, C2, FH3, FH4, LD1, LD2, Q1, Q2, Q3, Q4, R1, R10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

Commit message: Ready to send to production
Parts:
- added GL1: ~, DB_Logo_Footprints:Myscion_Dynamics_Main, symbol DB:Logos/Myscion Dynamics Yinglet Logo
Connections:
- net GND: now also J2.6 (Pin_6)
Other:
- note added: "If the proper fuses can not be found any fast 2512 fuses can be used instead."
- note added: "Replacement Fuses +15V 3.5A: 45303.5, 45103.5, 44803.5 +12V 0.4A 453.4, 451.4, 448.4 +5V 6.3A: 45306.3, 45106.3, 44806.3 -5V 0.08A: 453.08, 451.08, 448.08 -12V 0.1A: 453.1, 451.1, 448.1"
- moved on the sheet: C1, C2, C3, C4, C5, FH1, FH2, FH3, FH4, FH5, J1, J2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

Commit message: Sent PCB out to fab
Parts:
- added GL2: ~, Symbol:OSHW-Logo_11.4x12mm_SilkScreen, symbol DB:Logos/OSHW Logo
Other:
- note added: "+15V 3.5A: 45303.5, 45103.5, 44803.5 +12V 0.4A 453.4, 451.4, 448.4 +5V 6.3A: 45306.3, 45106.3, 44806.3 -5V 0.08A: 453.08, 451.08, 448.08 -12V 0.1A: 453.1, 451.1, 448.1"
- note added: "Replacement Fuses"
- note removed: "Replacement Fuses +15V 3.5A: 45303.5, 45103.5, 44803.5 +12V 0.4A 453.4, 451.4, 448.4 +5V 6.3A: 45306.3, 45106.3, 44806.3 -5V 0.08A: 453.08, 451.08, 448.08 -12V 0.1A: 453.1, 451.1, 448.1"
Changed lines of the file:
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@@
 	(text "If the proper fuses can not be found \nany fast 2512 fuses can be used instead."
 		(exclude_from_sim no)
-		(at 176.53 218.44 0)
+		(at 208.28 254 0)
 		(effects
 			(font
@@
 		)
 	)
+	(text "Replacement Fuses"
+		(exclude_from_sim no)
+		(at 189.23 227.33 0)
+		(effects
+			(font
+				(size 2.286 2.286)
+				(thickness 0.4572)
+				(bold yes)
+			)
+			(justify left)
+		)
+	)
 	(text "0.06 I2t\nFusing"
 		(exclude_from_sim no)
@@
 		)
 	)
-	(text "Replacement Fuses\n+15V 3.5A: 45303.5, 45103.5, 44803.5 \n+12V 0.4A 453.4, 451.4, 448.4\n+5V 6.3A: 45306.3, 45106.3, 44806.3\n-5V 0.08A: 453.08, 451.08, 448.08\n-12V 0.1A: 453.1, 451.1, 448.1\n"
+	(text "+15V 3.5A: 45303.5, 45103.5, 44803.5 \n+12V 0.4A 453.4, 451.4, 448.4\n+5V 6.3A: 45306.3, 45106.3, 44806.3\n-5V 0.08A: 453.08, 451.08, 448.08\n-12V 0.1A: 453.1, 451.1, 448.1\n"
 		(exclude_from_sim no)
-		(at 302.26 167.64 0)
+		(at 181.61 238.76 0)
 		(effects
 			(font
@@
 					(unit 1)
 				)
+			)
+		)
+	)
+	(symbol
+		(lib_id "DB:Logos/OSHW Logo")
+		(at 344.17 198.12 0)
+		(unit 1)
+		(exclude_from_sim no)
+		(in_bom no)
+		(on_board yes)
+		(dnp no)
+		(fields_autoplaced yes)
+		(property "Reference" "GL2"
+			(at 343.408 186.436 0)
+			(effects
+				(font
+					(size 1.27 1.27)
+				)
+				(hide yes)
+			)
+		)
+		(property "Value" "~"
+			(at 344.17 198.12 0)
+			(effects
+				(font
+					(size 1.27 1.27)
+				)
+				(hide yes)
+			)
+		)
+		(property "Footprint" "Symbol:OSHW-Logo_11.4x12mm_SilkScreen"
+			(at 344.17 198.12 0)
+			(effects
+				(font
+					(size 1.27 1.27)
+				)
+				(hide yes)
+			)
+		)
+		(property "Datasheet" ""
+			(at 344.17 198.12 0)
+			(effects
+				(font
+					(size 1.27 1.27)
+				)
+				(hide yes)
+			)
+		)
+		(property "Description" "OSHW Logo"
+			(at 344.17 198.12 0)
+			(effects
+				(font
+					(size 1.27 1.27)
+				)
+				(hide yes)
+			)
+		)
+		(property "Symbol Heritage" "NONE"
+			(at 344.17 198.12 0)
+			(effects
+				(font
+					(size 1.27 1.27)
+				)
+				(hide yes)
+			)
+		)
+		(property "Footprint Heritage" "NONE"
+			(at 344.17 198.12 0)
+			(effects
+				(font
+					(size 1.27 1.27)
+				)
+				(hide yes)
+			)
+		)
+		(instances
+			(project ""
+				(path "/ba2b9114-e1a5-46b3-b25b-16fdae1043bd"
+					(reference "GL2")
+					(unit 1)
+				)
